File: tests/Memory.sch (KiCad schematic (older format))
At the start: 8 parts, among them U5 16Mx16 SDRAM

Commit message: Added recursive operations on hierarchical schematics.
Parts:
- C10: footprint Capacitors_SMD:C_0603 -> G0jKWIb3lmifWK5; zzz4ozZ3f (none) -> ls8Y; zzz9xP (none) -> e6lpz2qKSOROTlUrJNt; zzzky (none) -> ze0MOSePdkElE
- C11: manf (none) -> Aqa5hLzPQbvEkrhj4PL; manf# (none) -> NsH3j
- C12: footprint Capacitors_SMD:C_0603 -> an97XYWHQ; manf# (none) -> 1IM9tfbull8Z
- C14: zzzkoq (none) -> 6kOG5onN96PhKO; zzzky (none) -> mTi4oVSHBX
- C8: value 0.1uF -> U2HOmXEe; zzz4ozZ3f (none) -> UymIG9gokKPJeZi6kCX
Changed lines of the file:
@@
 F 2 "XESS:TSOPII-54" H 5500 2500 60 0001 C CNN
 F 3 "" H 5500 2500 60 0000 C CNN
-F 4 "AS4C16M16S-6TCN" H 5500 2500 60 0001 C CNN "manf#"
-F 5 "Alliance Memory Inc." H 5500 2500 60 0001 C CNN "manf"
+F 4 "Alliance Memory Inc." H 5500 2500 60 0001 C CNN "manf"
+F 5 "AS4C16M16S-6TCN" H 5500 2500 60 0001 C CNN "manf#"
 	1    5500 2500
 	1    0    0    -1
@@
 F 0 "C12" H 6375 5850 50 0000 L CNN
 F 1 "0.1uF" H 6375 5650 50 0000 L CNN
-F 2 "Capacitors_SMD:C_0603" H 6388 5600 30 0001 C CNN
+F 2 "an97XYWHQ" H 6388 5600 30 0001 C CNN
 F 3 "" H 6350 5750 60 0000 C CNN
-F 4 "" H 0 0 50 0001 C CNN "manf#"
-F 5 "" H 0 0 50 0001 C CNN "manf"
+F 4 "1IM9tfbull8Z" H 0 0 50 0001 C CNN "manf#"
 	1    6350 5750
 	1    0    0    -1
@@
 F 2 "Capacitors_SMD:C_0603" H 6688 5600 30 0001 C CNN
 F 3 "" H 6650 5750 60 0000 C CNN
-F 4 "" H 0 0 50 0001 C CNN "manf#"
-F 5 "" H 0 0 50 0001 C CNN "manf"
 	1    6650 5750
 	1    0    0    -1
@@
 F 2 "Capacitors_SMD:C_0603" H 6988 5600 30 0001 C CNN
 F 3 "" H 6950 5750 60 0000 C CNN
-F 4 "" H 0 0 50 0001 C CNN "manf#"
-F 5 "" H 0 0 50 0001 C CNN "manf"
+F 4 "6kOG5onN96PhKO" H 0 0 50 0001 C CNN "zzzkoq"
+F 5 "mTi4oVSHBX" H 0 0 50 0001 C CNN "zzzky"
 	1    6950 5750
 	1    0    0    -1
@@
 P 5150 5750
 F 0 "C8" H 5175 5850 50 0000 L CNN
-F 1 "0.1uF" H 5175 5650 50 0000 L CNN
+F 1 "U2HOmXEe" H 5175 5650 50 0000 L CNN
 F 2 "Capacitors_SMD:C_0603" H 5188 5600 30 0001 C CNN
-F 3 "" H 5150 5750 60 0000 C CNN
+F 3 "bG3DDJhJEuZ73iP" H 5150 5750 60 0000 C CNN
 F 4 "GRM188R71C104KA01D" H 5150 5750 60 0001 C CNN "manf#"
-F 5 "" H 0 0 50 0001 C CNN "manf"
+F 5 "UymIG9gokKPJeZi6kCX" H 0 0 50 0001 C CNN "zzz4ozZ3f"
 	1    5150 5750
 	1    0    0    -1
@@
 F 2 "Capacitors_SMD:C_0603" H 5488 5600 30 0001 C CNN
 F 3 "" H 5450 5750 60 0000 C CNN
-F 4 "" H 0 0 50 0001 C CNN "manf#"
-F 5 "" H 0 0 50 0001 C CNN "manf"
 	1    5450 5750
 	1    0    0    -1
@@
 F 0 "C10" H 5775 5850 50 0000 L CNN
 F 1 "0.1uF" H 5775 5650 50 0000 L CNN
-F 2 "Capacitors_SMD:C_0603" H 5788 5600 30 0001 C CNN
+F 2 "G0jKWIb3lmifWK5" H 5788 5600 30 0001 C CNN
 F 3 "" H 5750 5750 60 0000 C CNN
-F 4 "" H 0 0 50 0001 C CNN "manf#"
-F 5 "" H 0 0 50 0001 C CNN "manf"
+F 4 "ls8Y" H 0 0 50 0001 C CNN "zzz4ozZ3f"
+F 5 "e6lpz2qKSOROTlUrJNt" H 0 0 50 0001 C CNN "zzz9xP"
+F 6 "ze0MOSePdkElE" H 0 0 50 0001 C CNN "zzzky"
 	1    5750 5750
 	1    0    0    -1
@@
 F 2 "Capacitors_SMD:C_0603" H 6088 5600 30 0001 C CNN
 F 3 "" H 6050 5750 60 0000 C CNN
-F 4 "" H 0 0 50 0001 C CNN "manf#"
-F 5 "" H 0 0 50 0001 C CNN "manf"
+F 4 "Aqa5hLzPQbvEkrhj4PL" H 0 0 50 0001 C CNN "manf"
+F 5 "NsH3j" H 0 0 50 0001 C CNN "manf#"
 	1    6050 5750
 	1    0    0    -1
